File: pcb/pocasicko.kicad_pcb (KiCad board)
At the start: 2 copper layers, 100 x 88 mm, 68 parts, among them J1 SMA, J2 Header_SMD_1x05, J3 FPC24, J4 Header_SMD_1x03, Q1 AO3400A, SW1 RESET, SW2 A, SW3 B, SW4 C, SW5 D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

Commit message: Exchanged FPC connector. This is the Rev. 1.
Parts:
- J3: footprint Moje:Waveshare_EPD_4.2_Amphenol_SFV24R-4STBE1HLF -> Moje:Waveshare_EPD_4.2_Molex_5034802400
Routing:
- net GND: track 152.5 -> 153.7 mm
